Commit message: motor standing fix

File: description/gazebo_control.xacro (robot description, xacro)
@@ -9,6 +9,6 @@
             <wheel_radius>0.05</wheel_radius>
             <!-- limits -->
-            <max_wheel_torque>200</max_wheel_torque>
-            <max_wheel_acceleration>10.0</max_wheel_acceleration>
+            <max_wheel_torque>20</max_wheel_torque>
+            <max_wheel_acceleration>2.0</max_wheel_acceleration>
             <!-- output -->
             <topic>cmd_vel</topic>

File: description/robot_core.xacro (robot description, xacro)
@@ -39,5 +39,5 @@
         </collision>
         <xacro:inertial_box mass="5" size="0.3 0.3 0.15">
-        <origin xyz="0.15 0 0.075" rpy="0 0 0"/>
+        <origin xyz="0.175 0 0.0" rpy="0 0 0"/>
         </xacro:inertial_box>
     </link>
